File: Kicad/Projetos/aracnobot/aracnobot.kicad_pcb (KiCad board)
At the start: 2 copper layers, 1 part, among them U1 SC0195_9_

Commit message: Kicad atualaizao footprint e schematico
Parts:
- added M1: Motor_Servo, Connector_PinHeader_2.54mm:PinHeader_1x03_P2.54mm_Vertical, F.Cu at (178.5, 69.0)
- added U2: DEVKIT_V1_ESP32-WROOM-32, DEVKIT_V1_ESP32-WROOM-32:MODULE_DEVKIT_V1_ESP32-WROOM-32, F.Cu at (153.8, 86.0)
