File: Kicad/Projetos/aracnobot/aracnobot.kicad_sch (KiCad schematic)
At the start: 1 part, among them U1 RASPBERRY_PI_3_MODEL_B_

Commit message: model 4 B
Parts:
- removed U1: RASPBERRY_PI_3_MODEL_B_, Raspberry_Pi_Footprints:MODULE_RASPBERRY_PI_3_MODEL_B_, symbol RASPBERRY_PI_3_MODEL_B_:RASPBERRY_PI_3_MODEL_B_
- added U1: SC0195_9_, Raspberry_pi_4_B:MODULE_SRASPBERRY_PI_4_MODEL_B_, symbol RASPBERRY_PI_4_MODEL_B_:SC0195_9_
Connections:
- net 3V3: now also U1.1 (3V3), U1.17 (3V3)
- net GND: now also U1.14 (GND), U1.20 (GND), U1.25 (GND), U1.30 (GND), U1.34 (GND), U1.39 (GND), U1.6 (GND), U1.9 (GND)
- net SHIELD: now also U1.S1 (SHIELD), U1.S2 (SHIELD), U1.S3 (SHIELD), U1.S4 (SHIELD)
- new net 5V0: U1.2 (5V0), U1.4 (5V0)
Changed lines of the file:
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@@
 	(paper "A4")
 	(symbol
-		(lib_id "RASPBERRY_PI_3_MODEL_B_:RASPBERRY_PI_3_MODEL_B_")
-		(at 137.16 93.98 0)
+		(lib_id "RASPBERRY_PI_4_MODEL_B_:SC0195_9_")
+		(at 129.54 87.63 0)
 		(unit 1)
 		(body_style 1)
@@
 		(fields_autoplaced yes)
 		(property "Reference" "U1"
-			(at 137.16 55.88 0)
-			(show_name no)
-			(do_not_autoplace no)
-			(effects
-				(font
-					(size 1.27 1.27)
-				)
-			)
-		)
-		(property "Value" "RASPBERRY_PI_3_MODEL_B_"
-			(at 137.16 58.42 0)
-			(show_name no)
-			(do_not_autoplace no)
-			(effects
-				(font
-					(size 1.27 1.27)
-				)
-			)
-		)
-		(property "Footprint" "Raspberry_Pi_Footprints:MODULE_RASPBERRY_PI_3_MODEL_B_"
-			(at 137.16 93.98 0)
+			(at 128.27 57.15 0)
+			(show_name no)
+			(do_not_autoplace no)
+			(effects
+				(font
+					(size 1.27 1.27)
+				)
+			)
+		)
+		(property "Value" "SC0195_9_"
+			(at 128.27 59.69 0)
+			(show_name no)
+			(do_not_autoplace no)
+			(effects
+				(font
+					(size 1.27 1.27)
+				)
+			)
+		)
+		(property "Footprint" "Raspberry_pi_4_B:MODULE_SRASPBERRY_PI_4_MODEL_B_"
+			(at 129.54 87.63 0)
 			(hide yes)
 			(show_name no)
@@
 		)
 		(property "Datasheet" ""
-			(at 137.16 93.98 0)
-			(hide yes)
-			(show_name no)
-			(do_not_autoplace no)
-			(effects
-				(font
-					(size 1.27 1.27)
-				)
-			)
-		)
-		(property "Description" "Single Board Computer, Model B+ 1GB RAM,Raspberry Pi 3 Series | Raspberry Pi RASPBERRY PI 3 MODEL B+"
-			(at 137.16 93.98 0)
+			(at 129.54 87.63 0)
+			(hide yes)
+			(show_name no)
+			(do_not_autoplace no)
+			(effects
+				(font
+					(size 1.27 1.27)
+				)
+			)
+		)
+		(property "Description" "The Raspberry Pi 4 Model B SC0195-9 single board computer features a powerful Broadcom BCM2711 ARM Cortex-A72 processor with 1.5GHz speed and four cores, making it ideal for demanding embedded computing applications. With 8GB of RAM and a compact size of 3.346 x 2.205, this SBC offers robust performance in a small footprint. It includes 40 digital I/O lines, GbE Ethernet, and multiple USB ports (two USB 2.0 and two USB 3.0), providing versatile connectivity options. Additionally, it supports video outputs such as CSI, DSI, and HDMI, making it suitable for a wide range of multimedia projects."
+			(at 129.54 87.63 0)
 			(hide yes)
 			(show_name no)
@@
 		)
 		(property "MF" "Raspberry Pi"
-			(at 137.16 93.98 0)
-			(hide yes)
-			(show_name no)
-			(do_not_autoplace no)
-			(effects
-				(font
-					(size 1.27 1.27)
-				)
-				(justify bottom)
-			)
-		)
-		(property "MAXIMUM_PACKAGE_HEIGHT" "16 mm"
-			(at 137.16 93.98 0)
-			(hide yes)
-			(show_name no)
-			(do_not_autoplace no)
-			(effects
-				(font
-					(size 1.27 1.27)
-				)
-				(justify bottom)
-			)
-		)
-		(property "Package" "Raspberry Pi"
-			(at 137.16 93.98 0)
+			(at 129.54 87.63 0)
+			(hide yes)
+			(show_name no)
+			(do_not_autoplace no)
+			(effects
+				(font
+					(size 1.27 1.27)
+				)
+				(justify bottom)
+			)
+		)
+		(property "Package" "None"
+			(at 129.54 87.63 0)
 			(hide yes)
 			(show_name no)
@@
 		)
 		(property "Price" "None"
-			(at 137.16 93.98 0)
-			(hide yes)
-			(show_name no)
-			(do_not_autoplace no)
-			(effects
-				(font
-					(size 1.27 1.27)
-				)
-				(justify bottom)
-			)
-		)
-		(property "Check_prices" "https://www.snapeda.com/parts/RASPBERRY%20PI%203%20MODEL%20B+/Raspberry+Pi/view-part/?ref=eda"
-			(at 137.16 93.98 0)
+			(at 129.54 87.63 0)
+			(hide yes)
+			(show_name no)
+			(do_not_autoplace no)
+			(effects
+				(font
+					(size 1.27 1.27)
+				)
+				(justify bottom)
+			)
+		)
+		(property "Check_prices" "https://www.snapeda.com/parts/SC0195(9)/Raspberry+Pi/view-part/?ref=eda"
+			(at 129.54 87.63 0)
+			(hide yes)
+			(show_name no)
+			(do_not_autoplace no)
+			(effects
+				(font
+					(size 1.27 1.27)
+				)
+				(justify bottom)
+			)
+		)
+		(property "MAXIMUM_PACKAGE_HIEGHT" "18mm"
+			(at 129.54 87.63 0)
 			(hide yes)
 			(show_name no)
@@
 		)
 		(property "STANDARD" "Manufacturer Recommendations"
-			(at 137.16 93.98 0)
-			(hide yes)
-			(show_name no)
-			(do_not_autoplace no)
-			(effects
-				(font
-					(size 1.27 1.27)
-				)
-				(justify bottom)
-			)
-		)
-		(property "PARTREV" "N/A"
-			(at 137.16 93.98 0)
-			(hide yes)
-			(show_name no)
-			(do_not_autoplace no)
-			(effects
-				(font
-					(size 1.27 1.27)
-				)
-				(justify bottom)
-			)
-		)
-		(property "SnapEDA_Link" "https://www.snapeda.com/parts/RASPBERRY%20PI%203%20MODEL%20B+/Raspberry+Pi/view-part/?ref=snap"
-			(at 137.16 93.98 0)
-			(hide yes)
-			(show_name no)
-			(do_not_autoplace no)
-			(effects
-				(font
-					(size 1.27 1.27)
-				)
-				(justify bottom)
-			)
-		)
-		(property "MP" "RASPBERRY PI 3 MODEL B+"
-			(at 137.16 93.98 0)
-			(hide yes)
-			(show_name no)
-			(do_not_autoplace no)
-			(effects
-				(font
-					(size 1.27 1.27)
-				)
-				(justify bottom)
-			)
-		)
-		(property "SNAPEDA_PN" "RASPBERRY PI 3 MODEL B+"
-			(at 137.16 93.98 0)
+			(at 129.54 87.63 0)
+			(hide yes)
+			(show_name no)
+			(do_not_autoplace no)
+			(effects
+				(font
+					(size 1.27 1.27)
+				)
+				(justify bottom)
+			)
+		)
+		(property "PARTREV" "1.0"
+			(at 129.54 87.63 0)
+			(hide yes)
+			(show_name no)
+			(do_not_autoplace no)
+			(effects
+				(font
+					(size 1.27 1.27)
+				)
+				(justify bottom)
+			)
+		)
+		(property "SnapEDA_Link" "https://www.snapeda.com/parts/SC0195(9)/Raspberry+Pi/view-part/?ref=snap"
+			(at 129.54 87.63 0)
+			(hide yes)
+			(show_name no)
+			(do_not_autoplace no)
+			(effects
+				(font
+					(size 1.27 1.27)
+				)
+				(justify bottom)
+			)
+		)
+		(property "MP" "SC0195(9)"
+			(at 129.54 87.63 0)
 			(hide yes)
 			(show_name no)
@@
 		)
 		(property "Availability" "In Stock"
-			(at 137.16 93.98 0)
+			(at 129.54 87.63 0)
 			(hide yes)
 			(show_name no)
@@
 		)
 		(property "MANUFACTURER" "Raspberry Pi"
-			(at 137.16 93.98 0)
-			(hide yes)
-			(show_name no)
-			(do_not_autoplace no)
-			(effects
-				(font
-					(size 1.27 1.27)
-				)
-				(justify bottom)
-			)
+			(at 129.54 87.63 0)
+			(hide yes)
+			(show_name no)
+			(do_not_autoplace no)
+			(effects
+				(font
+					(size 1.27 1.27)
+				)
+				(justify bottom)
+			)
+		)
+		(pin "10"
+		)
+		(pin "11"
+		)
+		(pin "9"
+		)
+		(pin "7"
+		)
+		(pin "6"
+		)
+		(pin "5"
+		)
+		(pin "4"
+		)
+		(pin "3"
+		)
+		(pin "2"
+		)
+		(pin "1"
 		)
 		(pin "8"
 		)
-		(pin "7"
-		)
-		(pin "6"
-		)
-		(pin "5"
-		)
-		(pin "4"
-		)
-		(pin "3"
-		)
-		(pin "2"
-		)
-		(pin "1"
-		)
-		(pin "9"
-		)
-		(pin "10"
-		)
-		(pin "11"
-		)
 		(pin "12"
 		)
@@
 		(pin "40"
 		)
-		(pin "41"
-		)
-		(pin "42"
-		)
-		(pin "43"
-		)
-		(pin "44"
-		)
 		(pin "S1"
